Commit message: Depth Camera and Camera Working

File: description/lidar.xacro (robot description, xacro)
@@ -26,6 +26,7 @@
     <!-- Gazebo stuff -->
     <gazebo reference="laser_frame">
+        <material>Gazebo/Red</material>
         <!-- Simulatefd Sensors -->
-        <sensor name="name" type="ray">
+        <sensor name="lidar" type="ray">
             <pose> 0 0 0 0 0 0 </pose>
             <visualize>true</visualize>
@@ -49,7 +50,7 @@
                 <ros>
                     <!-- Had an error with the argument tag -->
-                    <!-- <argument>~/out:=scan</argument> -->
-                    <namespace>/</namespace>
-                    <remapping>~/scan:=scan</remapping>
+                    <argument>~/out:=scan</argument>
+                    <!-- <namespace>/</namespace> -->
+                    <!-- <remapping>~/scan:=scan</remapping> -->
                 </ros>
                 <output_type>sensor_msgs/LaserScan</output_type>

File: description/robot.urdf.xacro (robot description, xacro)
@@ -5,3 +5,4 @@
     <xacro:include filename="lidar.xacro"/>
     <!-- <xacro:include filename="camera.xacro"/> -->
+    <xacro:include filename="depth_camera.xacro"/>
 </robot>
